File: hw/uavprobe/connectors.kicad_sch (KiCad schematic)
At the start: 0 parts

Commit message: Connectors sheet and CAN/ESD
Parts:
- added C17, C18, C19, C20, C21, C22, C23, C24, C25, C26, C27, C28: 1u, symbol Device:C
- added J1: 6-pin A, symbol Connector_Generic_MountingPin:Conn_01x06_MountingPin
- added J10: I^{2}C, symbol Connector_Generic_MountingPin:Conn_01x04_MountingPin
- added J11: SERIAL2, symbol Connector_Generic_MountingPin:Conn_01x04_MountingPin
- added J12: USB2, symbol Connector_Generic_MountingPin:Conn_01x04_MountingPin
- added J13: CAN1, symbol Connector_Generic_MountingPin:Conn_01x04_MountingPin
- added J14: CAN2, symbol Connector_Generic_MountingPin:Conn_01x04_MountingPin
- added J15: SERIAL1 (Lidar), symbol Connector_Generic_MountingPin:Conn_01x04_MountingPin
- added J16: I^{2}C (Lidar), symbol Connector_Generic_MountingPin:Conn_01x04_MountingPin
- added J2: 6-pin B, symbol Connector_Generic_MountingPin:Conn_01x06_MountingPin
- added J3: 4-pin A, symbol Connector_Generic_MountingPin:Conn_01x04_MountingPin
- added J4: 4-pin B, symbol Connector_Generic_MountingPin:Conn_01x04_MountingPin
- added J5: SERIAL1, symbol Connector_Generic_MountingPin:Conn_01x04_MountingPin
- added J6: SERIAL1/2, symbol Connector_Generic_MountingPin:Conn_01x06_MountingPin
- added J7: SERIAL1 (flow control), symbol Connector_Generic_MountingPin:Conn_01x06_MountingPin
- added J8: SERIAL2/1, symbol Connector_Generic_MountingPin:Conn_01x06_MountingPin
- added J9: SERIAL1 (GPS/I2C), symbol Connector_Generic_MountingPin:Conn_01x06_MountingPin
Connections:
- new net: J3.1 (Pin_1), J4.1 (Pin_1)
- new net: J3.2 (Pin_2), J4.2 (Pin_2)
- new net: J3.3 (Pin_3), J4.3 (Pin_3)
- new net: J3.4 (Pin_4), J4.4 (Pin_4)
- new net: C27.1, J15.3 (Pin_3)
- new net: J1.1 (Pin_1), J2.1 (Pin_1)
- new net: J1.2 (Pin_2), J2.2 (Pin_2)
- new net: J1.3 (Pin_3), J2.3 (Pin_3)
- new net: J1.4 (Pin_4), J2.4 (Pin_4)
- new net: J1.5 (Pin_5), J2.5 (Pin_5)
- new net: J1.6 (Pin_6), J2.6 (Pin_6)
- new net: C28.1, J16.3 (Pin_3)
- new net CAN1_D+: J13.2 (Pin_2)
- new net CAN1_D-: J13.3 (Pin_3)
- new net CAN2_D+: J14.2 (Pin_2)
- new net CAN2_D-: J14.3 (Pin_3)
- new net GND: C17.1, C17.2, C18.1, C18.2, C19.1, C19.2, C20.1, C20.2, C21.1, C21.2, C22.1, C22.2, C23.1, C23.2, C24.1, C24.2, C25.1, C25.2, C26.1, C26.2, C27.2, C28.2, J10.1 (Pin_1), J10.4 (Pin_4), J10.MP (MountPin), J11.1 (Pin_1), J11.4 (Pin_4), J11.MP (MountPin), J12.1 (Pin_1), J12.4 (Pin_4), J12.MP (MountPin), J13.1 (Pin_1), J13.4 (Pin_4), J13.MP (MountPin), J14.1 (Pin_1), J14.4 (Pin_4), J14.MP (MountPin), J15.4 (Pin_4), J15.MP (MountPin), J16.4 (Pin_4), J16.MP (MountPin), J5.1 (Pin_1), J5.4 (Pin_4), J5.MP (MountPin), J6.1 (Pin_1), J6.6 (Pin_6), J6.MP (MountPin), J7.1 (Pin_1), J7.6 (Pin_6), J7.MP (MountPin), J8.1 (Pin_1), J8.6 (Pin_6), J8.MP (MountPin), J9.1 (Pin_1), J9.6 (Pin_6), J9.MP (MountPin)
- new net I2C_SCL: J10.2 (Pin_2), J16.1 (Pin_1), J9.4 (Pin_4)
- new net I2C_SDA: J10.3 (Pin_3), J16.2 (Pin_2), J9.5 (Pin_5)
- new net UART1_CTS: J7.4 (Pin_4)
- new net UART1_RTS: J7.5 (Pin_5)
- new net UART1_RX: J15.2 (Pin_2), J5.3 (Pin_3), J6.3 (Pin_3), J7.3 (Pin_3), J8.4 (Pin_4), J9.3 (Pin_3)
- new net UART1_TX: J15.1 (Pin_1), J5.2 (Pin_2), J6.2 (Pin_2), J7.2 (Pin_2), J8.5 (Pin_5), J9.2 (Pin_2)
- new net UART2_RX: J11.3 (Pin_3), J6.5 (Pin_5), J8.2 (Pin_2)
- new net UART2_TX: J11.2 (Pin_2), J6.4 (Pin_4), J8.3 (Pin_3)
- new net USB2_D+: J12.3 (Pin_3)
- new net USB2_D-: J12.2 (Pin_2)
- no-connect marks 0 -> 4
Other:
- note added: "Benewake Lidar"
- note added: "CAN"
- note added: "I^{2}C"
- note added: "NOTE: TX/RX reversed in order to connect with SERIAL1/2 and and form a 2-UART loopback"
- note added: "Pass-through (Unconnected)"
- note added: "Serial (Combined)"
- note added: "Serial UART"
- note added: "USB"

Commit message: USB sheet
Parts:
- C24: value 1u -> 10u
Connections:
- net GND: no longer C24.1, J12.1 (Pin_1)
- new net VBUS2: C24.1, J12.1 (Pin_1)

Commit message: Cleanup and root sheet
Parts:
- renumbered C17 to C27, C18 to C28, C19 to C29, C20 to C30, C21 to C31, C22 to C32, C27 to C33, C28 to C34, C23 to C35, C24 to C36, C25 to C37, C26 to C38, J7 to J10, J9 to J11, J15 to J12, J16 to J13, J10 to J14, J12 to J15, J13 to J16, J14 to J17, J1 to J2, J5 to J4, J11 to J5, J8 to J7, J2 to J8, J4 to J9

Commit message: ERC pass
Footprint and symbol copy editing warnings left
Parts:
- removed C34: 1u, symbol Device:C
- added C36: 1u, symbol Device:C
- renumbered C27 to C29, C28 to C30, C29 to C31, C30 to C32, C31 to C33, C32 to C34, C33 to C35, C35 to C37, C36 to C38, C37 to C39, C38 to C40
Connections:
- net GND: now also C35.1, C36.1; no longer C29.1, C30.1, C31.1, C32.1, C33.1, C34.1, C35.2, C37.1, C39.1, C40.1, J10.1 (Pin_1), J11.1 (Pin_1), J14.1 (Pin_1), J16.1 (Pin_1), J17.1 (Pin_1), J4.1 (Pin_1), J5.1 (Pin_1), J6.1 (Pin_1), J7.1 (Pin_1)
- net VBUS: now reaches J12.3 (Pin_3)
- net VBUS: now also C29.1, C30.1, C31.1, C32.1, C33.1, C34.1, C35.2, C37.1, C39.1, C40.1, J10.1 (Pin_1), J11.1 (Pin_1), J13.3 (Pin_3), J14.1 (Pin_1), J16.1 (Pin_1), J17.1 (Pin_1), J4.1 (Pin_1), J5.1 (Pin_1), J6.1 (Pin_1), J7.1 (Pin_1), C36.2; no longer C35.1
Other:
- moved on the sheet: C35

Commit message: Footprint/MPN assignment pass
Parts:
- C29, C30, C31, C32, C33, C34, C35, C36, C37, C38, C39, C40: footprint (none) -> Capacitor_SMD:C_0402_1005Metric
- J10, J11, J2, J6, J7, J8: footprint (none) -> Connector_JST:JST_GH_BM06B-GHS-TBT_1x06-1MP_P1.25mm_Vertical; MPN (none) -> BM06B-GHS-TBT
- J12, J13, J14, J15, J16, J17, J3, J4, J5, J9: footprint (none) -> Connector_JST:JST_GH_BM04B-GHS-TBT_1x04-1MP_P1.25mm_Vertical; MPN (none) -> BM04B-GHS-TBT

Commit message: Layout revision 1
Pre-DRC
Parts:
- J10: value SERIAL1 (flow control) -> SERIAL1 (flow)
Changed lines of the file:
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@@
 			)
 		)
-		(property "Value" "SERIAL1 (flow control)"
+		(property "Value" "SERIAL1 (flow)"
 			(at 100.33 39.7255 0)
 			(effects
